File: PCB/LED Chaser.kicad_pcb (KiCad board)
At the start: 2 copper layers, 60 x 51.2 mm, 19 parts, among them J1 Conn_01x03_Pin, U1 NE555P, U2 4017

Commit message: modified back silkscreen
Other:
- board text added: "L.Z. 12/25"
- board text removed: "L.Z. 12/25 ILY <3"
Changed lines of the file:
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@@
 		)
 	)
-	(gr_text "L.Z.\n12/25\nILY <3"
+	(gr_text "L.Z.\n12/25"
 		(at 133.005 48 0)
 		(layer "B.SilkS")
